File: ESP32-C6 USB switch.kicad_sch (KiCad schematic)
At the start: 0 parts

Commit message: wired HUSB237 and 20V5A type-C port together
Parts:
- added C1: 20nF, symbol Device:C_Small
- added C2: 1uF, symbol Device:C_Small
- added U1: HUSB237-AA001-DN06R, JLCImport:HUSB237-AA001-DN06R, symbol JLCImport:HUSB237-AA001-DN06R
- added USB1, USB2: TYPE-C-31-M-31, JLCImport:TYPE-C-31-M-31, symbol JLCImport:TYPE-C-31-M-31
Connections:
- new net: C1.1, U1.3 (VSET)
- new net GND: C1.2, C2.2, U1.7 (GND), USB1.1, USB1.A1 (GND), USB1.A12 (GND)
- new net IN_CC1: U1.1 (CC1), USB1.A5 (CC1)
- new net IN_CC2: U1.6 (CC2), USB1.B5 (CC2)
- new net IN_D+: U1.4 (D+), USB1.A6 (DP1), USB1.B6 (DP2)
- new net IN_D-: U1.5 (D-), USB1.A7 (DN1), USB1.B7 (DN2)
- new net IN_VBUS: C2.1, U1.2 (VUSB), USB1.A4 (VBUS), USB1.A9 (VBUS)
- no-connect marks 0 -> 2
